File: kicad/blinky.sch (KiCad schematic (older format))
At the start: 15 parts, among them Q1 MMBT2222, Q2 MMBT2222, Q3 MMBT2222, Q4 MMBT2222

Commit message: routing done
Parts:
- Q1, Q2, Q3, Q4: footprint Housings_SOT-23_SOT-143_TSOT-6:SOT-23 -> bb:SOT-23
Connections:
- net VCC: now reaches BT1.1, D1.2 (A), D2.2 (A), R3.1, R4.1, TP1.1
Changed lines of the file:
@@
 F 0 "Q1" H 3950 5225 50  0000 L CNN
 F 1 "MMBT2222" H 3950 5150 50  0000 L CNN
-F 2 "Housings_SOT-23_SOT-143_TSOT-6:SOT-23" H 3950 5075 50  0000 L CIN
+F 2 "bb:SOT-23" H 3950 5075 50  0000 L CIN
 F 3 "" H 3750 5150 50  0000 L CNN
 	1    3750 5150
@@
 $EndComp
 $Comp
-L Battery BT1
-U 1 1 55E27575
-P 2600 3850
-F 0 "BT1" H 2700 3900 50  0000 L CNN
-F 1 "Battery" H 2700 3800 50  0000 L CNN
-F 2 "bb:CR2032-SMD" V 2600 3890 60  0001 C CNN
-F 3 "" V 2600 3890 60  0000 C CNN
-	1    2600 3850
-	1    0    0    -1
-$EndComp
-$Comp
 L BC547 Q3
 U 1 1 55E2771E
@@
 F 0 "Q3" H 5400 4375 50  0000 L CNN
 F 1 "MMBT2222" H 5400 4300 50  0000 L CNN
-F 2 "Housings_SOT-23_SOT-143_TSOT-6:SOT-23" H 5400 4225 50  0000 L CIN
+F 2 "bb:SOT-23" H 5400 4225 50  0000 L CIN
 F 3 "" H 5200 4300 50  0000 L CNN
 	1    5200 4300
@@
 F 0 "Q4" H 7000 4375 50  0000 L CNN
 F 1 "MMBT2222" H 7000 4300 50  0000 L CNN
-F 2 "Housings_SOT-23_SOT-143_TSOT-6:SOT-23" H 7000 4225 50  0000 L CIN
+F 2 "bb:SOT-23" H 7000 4225 50  0000 L CIN
 F 3 "" H 6800 4300 50  0000 L CNN
 	1    6800 4300
@@
 F 0 "Q2" H 4750 5425 50  0000 L CNN
 F 1 "MMBT2222" H 4750 5350 50  0000 L CNN
-F 2 "Housings_SOT-23_SOT-143_TSOT-6:SOT-23" H 4750 5275 50  0000 L CIN
+F 2 "bb:SOT-23" H 4750 5275 50  0000 L CIN
 F 3 "" H 4550 5350 50  0000 L CNN
 	1    4550 5350
@@
 	4650 4800 4650 5150
 Wire Wire Line
-	2600 3700 2600 2400
-Wire Wire Line
-	2600 2400 6900 2400
+	2600 2300 2600 3700
 Wire Wire Line
 	5100 2400 5100 2600
@@
 Connection ~ 5700 3900
 Wire Wire Line
-	6300 3300 6300 2400
+	6300 2400 6300 3300
 Connection ~ 6300 2400
 Wire Wire Line
@@
 Wire Wire Line
 	3300 4375 3300 4600
+Wire Wire Line
+	2600 2400 6900 2400
+Connection ~ 2600 2400
+Text GLabel 2600 2300 1    60   Input ~ 0
+VCC
+$Comp
+L Battery BT1
+U 1 1 55E6B2B2
+P 2600 3850
+F 0 "BT1" H 2700 3900 50  0000 L CNN
+F 1 "Battery" H 2700 3800 50  0000 L CNN
+F 2 "bb:CR2032-SMD" V 2600 3890 60  0001 C CNN
+F 3 "" V 2600 3890 60  0000 C CNN
+	1    2600 3850
+	1    0    0    -1
+$EndComp
 $EndSCHEMATC

Commit message: switched to 1206 LEDs
Parts:
- D1, D2: footprint bb:MADW__PLCC2-3528 -> bb:LED-1206
Changed lines of the file:
@@
 F 0 "D1" H 5100 2900 50  0000 C CNN
 F 1 "LED" H 5100 2700 50  0000 C CNN
-F 2 "bb:MADW__PLCC2-3528" H 5100 2800 60  0001 C CNN
+F 2 "bb:LED-1206" H 5100 2800 60  0001 C CNN
 F 3 "" H 5100 2800 60  0000 C CNN
 	1    5100 2800
@@
 F 0 "D2" H 6900 2900 50  0000 C CNN
 F 1 "LED" H 6900 2700 50  0000 C CNN
-F 2 "bb:MADW__PLCC2-3528" H 6900 2800 60  0001 C CNN
+F 2 "bb:LED-1206" H 6900 2800 60  0001 C CNN
 F 3 "" H 6900 2800 60  0000 C CNN
 	1    6900 2800

Commit message: updated
Parts:
- Q1, Q2, Q3, Q4: footprint bb:SOT-23 -> bb:SOT-23_Handsoldering
Changed lines of the file:
@@
 F 0 "Q1" H 3950 5225 50  0000 L CNN
 F 1 "MMBT2222" H 3950 5150 50  0000 L CNN
-F 2 "bb:SOT-23" H 3950 5075 50  0000 L CIN
+F 2 "bb:SOT-23_Handsoldering" H 3950 5075 50  0001 L CIN
 F 3 "" H 3750 5150 50  0000 L CNN
 	1    3750 5150
@@
 F 0 "Q3" H 5400 4375 50  0000 L CNN
 F 1 "MMBT2222" H 5400 4300 50  0000 L CNN
-F 2 "bb:SOT-23" H 5400 4225 50  0000 L CIN
+F 2 "bb:SOT-23_Handsoldering" H 5400 4225 50  0001 L CIN
 F 3 "" H 5200 4300 50  0000 L CNN
 	1    5200 4300
@@
 F 0 "Q4" H 7000 4375 50  0000 L CNN
 F 1 "MMBT2222" H 7000 4300 50  0000 L CNN
-F 2 "bb:SOT-23" H 7000 4225 50  0000 L CIN
+F 2 "bb:SOT-23_Handsoldering" H 7000 4225 50  0001 L CIN
 F 3 "" H 6800 4300 50  0000 L CNN
 	1    6800 4300
@@
 F 0 "Q2" H 4750 5425 50  0000 L CNN
 F 1 "MMBT2222" H 4750 5350 50  0000 L CNN
-F 2 "bb:SOT-23" H 4750 5275 50  0000 L CIN
+F 2 "bb:SOT-23_Handsoldering" H 4750 5275 50  0001 L CIN
 F 3 "" H 4550 5350 50  0000 L CNN
 	1    4550 5350
